Commit message: Robot_body_issue_fixed

File: src/aurdinorobot_description/urdf/arduinorobot.urdf.xacro (robot description, xacro)
@@ -7,8 +7,8 @@
         <inertial>
             <mass value ="${mass}"/>
-            <inertial ixx= "1.0" ixy = "0.0" ixz = "0.0"
-            iyy = "1.0" iyz = "0.0"
-            izz = "1.0"/>
-        </inertial>
+            <inertia ixx="1.0" ixy = "0.0" ixz = "0.0"
+                      iyy="1.0" iyz = "0.0"
+                      izz="1.0"/>
+            </inertial>
     </xacro:macro>
     <link name= "world"/>
@@ -166,4 +166,5 @@
     </joint>
     <link name="rgb_camera">
+        <xacro:default_inertial mass = "0.001"/>
         <visual>
             <origin rpy="-1.57 0 -1.57" xyz="-0.1 0.125 0.15"/>
@@ -172,4 +173,10 @@
             </geometry>
         </visual>
+        <collision>
+            <origin rpy="-1.57 0 -1.57" xyz="-0.1 0.125 0.15"/>
+            <geometry>
+                <mesh filename="package://aurdinorobot_description/meshes/pi_camera.STL" scale="0.01 0.01 0.01"/>
+            </geometry>
+        </collision>
     </link>
     <joint name ="rgb_camera_joint" type="fixed">
