Commit message: controller_setup

File: install/aurdinorobot_description/share/aurdinorobot_description/urdf/arduinorobot.urdf.xacro (robot description, xacro)
@@ -1,4 +1,6 @@
 <?xml version="1.0"?>
 <robot xmlns:xacro = "http://www.ros.org/wiki/xacro" name = "aurdinorobot">
+    <xacro:include filename="$(find aurdinorobot_description)/urdf/arduinorobot_gazebo.xacro"/>
+    <xacro:include filename="$(find aurdinorobot_description)/urdf/arduinorobot_ros2_control.xacro"/>
     <xacro:property name="PI" value="3.14159"/>
     <xacro:property name="effort" value="30.0"/>
@@ -7,8 +9,17 @@
         <inertial>
             <mass value ="${mass}"/>
-            <inertial ixx= "1.0" ixy = "0.0" ixz = "0.0"
-            iyy = "1.0" iyz = "0.0"
-            izz = "1.0"/>
-        </inertial>
+            <inertia ixx="1.0" ixy = "0.0" ixz = "0.0"
+                      iyy="1.0" iyz = "0.0"
+                      izz="1.0"/>
+            </inertial>
+    </xacro:macro>
+    <xacro:macro name = "default_transmission" params = "number">
+        <transmission name = "transmission_${number}">
+            <plugin>transmission_interface/SimpleTransmission</plugin>
+            <actuator name = "motor_${number}" role = "actuator"/>
+            <joint name = "joint_${number}" role = "joint1">
+                <mechanical_reduction>1.0</mechanical_reduction>
+            </joint>
+        </transmission>
     </xacro:macro>
     <link name= "world"/>
@@ -166,4 +177,5 @@
     </joint>
     <link name="rgb_camera">
+        <xacro:default_inertial mass = "0.001"/>
         <visual>
             <origin rpy="-1.57 0 -1.57" xyz="-0.1 0.125 0.15"/>
@@ -172,4 +184,10 @@
             </geometry>
         </visual>
+        <collision>
+            <origin rpy="-1.57 0 -1.57" xyz="-0.1 0.125 0.15"/>
+            <geometry>
+                <mesh filename="package://aurdinorobot_description/meshes/pi_camera.STL" scale="0.01 0.01 0.01"/>
+            </geometry>
+        </collision>
     </link>
     <joint name ="rgb_camera_joint" type="fixed">
@@ -178,3 +196,7 @@
         <origin xyz="0 0.45 0.2" rpy="0 -0.5 1.57"/>
     </joint>
+    <xacro:default_transmission number="1"/>
+    <xacro:default_transmission number="2"/>
+    <xacro:default_transmission number="3"/>
+    <xacro:default_transmission number="4"/>
 </robot>

File: src/aurdinorobot_description/urdf/arduinorobot.urdf.xacro (robot description, xacro)
@@ -1,4 +1,6 @@
 <?xml version="1.0"?>
 <robot xmlns:xacro = "http://www.ros.org/wiki/xacro" name = "aurdinorobot">
+    <xacro:include filename="$(find aurdinorobot_description)/urdf/arduinorobot_gazebo.xacro"/>
+    <xacro:include filename="$(find aurdinorobot_description)/urdf/arduinorobot_ros2_control.xacro"/>
     <xacro:property name="PI" value="3.14159"/>
     <xacro:property name="effort" value="30.0"/>
@@ -12,4 +14,13 @@
             </inertial>
     </xacro:macro>
+    <xacro:macro name = "default_transmission" params = "number">
+        <transmission name = "transmission_${number}">
+            <plugin>transmission_interface/SimpleTransmission</plugin>
+            <actuator name = "motor_${number}" role = "actuator"/>
+            <joint name = "joint_${number}" role = "joint1">
+                <mechanical_reduction>1.0</mechanical_reduction>
+            </joint>
+        </transmission>
+    </xacro:macro>
     <link name= "world"/>
     <link name = "base_link">
@@ -185,3 +196,7 @@
         <origin xyz="0 0.45 0.2" rpy="0 -0.5 1.57"/>
     </joint>
+    <xacro:default_transmission number="1"/>
+    <xacro:default_transmission number="2"/>
+    <xacro:default_transmission number="3"/>
+    <xacro:default_transmission number="4"/>
 </robot>
